Commit message: Fix issues in differents files.

File: urdf/robaka_v2.xacro (robot description, xacro)
@@ -38,5 +38,4 @@
   </xacro:macro>
   <link name="base_footprint">
-    <xacro:box_inertia m="8" w="0.001" h="0.001" d="0.001"/>
     <visual>
       <origin xyz="0 0 0" rpy="0 0 0" />
@@ -75,5 +74,5 @@
     <link name="${prefix}_wheel">
       <visual>
-	<material name="darkgray"/>
+	      <material name="darkgray"/>
         <origin xyz="0 0 0" rpy="${pi/2} 0 0"/>
         <geometry>
@@ -120,5 +119,5 @@
     <xacro:sphere_inertia m="5" r="${caster_wheel_radius}"/>
   </link>
-  <joint name="caster_wheel_joint" type="continuous">
+  <joint name="caster_wheel_joint" type="fixed">
     <axis xyz="0 1 0" rpy="0 0 0" />
     <parent link="base_link"/>
@@ -153,3 +152,29 @@
   <link name="camera" type="fixed">
   </link>
+<gazebo reference="left_wheel">
+  <mu1>1.0</mu1>
+  <mu2>1.0</mu2>
+  <kp>1000000.0</kp>
+  <kd>100.0</kd>
+  <!-- -minDepth: Distance at which the wheel can insert under the floor.
+  For more information you can see http://osrf-distributions.s3.amazonaws.com/gazebo/api/1.6.3/classgazebo_1_1physics_1_1SurfaceParams.html#a648279b02a66224e3bbb361784e2964a -->
+  <minDepth>0.0001</minDepth>
+  <maxVel>1.0</maxVel>
+</gazebo>
+<gazebo reference="right_wheel">
+  <mu1>1.0</mu1>
+  <mu2>1.0</mu2>
+  <kp>1000000.0</kp>
+  <kd>100.0</kd>
+  <!-- -minDepth: Distance at which the wheel can insert under the floor.
+  For more information you can see http://osrf-distributions.s3.amazonaws.com/gazebo/api/1.6.3/classgazebo_1_1physics_1_1SurfaceParams.html#a648279b02a66224e3bbb361784e2964a -->
+  <minDepth>0.0001</minDepth>
+  <maxVel>1.0</maxVel>
+</gazebo>
+<gazebo reference="caster_wheel">
+  <mu1>0.1</mu1>
+  <mu2>0.1</mu2>
+  <kp>1000000.0</kp>
+  <kd>1.0</kd>
+</gazebo>
 </robot>

Commit message: change urdf.

File: urdf/robaka_v2.xacro (robot description, xacro)
@@ -75,13 +75,13 @@
       <visual>
 	      <material name="darkgray"/>
-        <origin xyz="0 0 0" rpy="${pi/2} 0 0"/>
-        <geometry>
-          <cylinder radius="${wheel_radius}" length="0.02"/>
+        <geometry>
+          <cylinder radius="${wheel_radius}" length="0.02"/>
+          <origin xyz="0 0 0" rpy="${pi/2} 0 0"/>
         </geometry>
       </visual>
       <collision>
-        <origin xyz="0 0 0" rpy="${pi/2} 0 0"/>
-        <geometry>
-          <cylinder radius="${wheel_radius}" length="0.02"/>
+        <geometry>
+          <cylinder radius="${wheel_radius}" length="0.02"/>
+          <origin xyz="0 0 0" rpy="${pi/2} 0 0"/>
         </geometry>
       </collision>
@@ -95,6 +95,43 @@
     </joint>
   </xacro:macro>
-  <xacro:wheel prefix="left" reflect="1"/>
-  <xacro:wheel prefix="right" reflect="-1"/>
+    <link name="right_wheel">
+      <visual>
+        <geometry>
+          <cylinder radius="${wheel_radius}" length="0.02"/>
+        </geometry>
+      </visual>
+      <collision>
+        <geometry>
+          <cylinder radius="${wheel_radius}" length="0.02"/>
+        </geometry>
+      </collision>
+      <xacro:cylinder_inertia m="10" r="${wheel_radius}" h="0.02"/>
+    </link>
+    <joint name="right_wheel_joint" type="continuous">
+      <axis xyz="0 1 0" rpy="0 0 0" />
+      <parent link="base_link"/>
+      <child link="right_wheel"/>
+      <origin xyz="${wheel_joint_offset} ${-((base_width/2)+base_wheel_gap)} -0.06" rpy="${pi/2} 0 0"/>
+    </joint>
+    <!-- Left -->
+    <joint name="left_wheel_joint" type="continuous">
+      <axis xyz="0 1 0" rpy="0 0 0" />
+      <parent link="base_link"/>
+      <child link="left_wheel"/>
+      <origin xyz="${wheel_joint_offset} ${((base_width/2)+base_wheel_gap)} -0.06" rpy="${pi/2} 0 0"/>
+    </joint>
+    <link name="left_wheel">
+      <visual>
+        <geometry>
+          <cylinder radius="${wheel_radius}" length="0.02"/>
+        </geometry>
+      </visual>
+      <collision>
+        <geometry>
+          <cylinder radius="${wheel_radius}" length="0.02"/>
+        </geometry>
+      </collision>
+      <xacro:cylinder_inertia m="10" r="${wheel_radius}" h="0.02"/>
+    </link>
   <xacro:macro name="sphere_inertia" params="m r">
     <inertial>
@@ -106,5 +143,4 @@
      <visual>
        <material name="darkgray"/>
-      <origin xyz="0 0 0" rpy="0 0 0"/>
       <geometry>
         <sphere radius="${caster_wheel_radius}"/>
@@ -112,5 +148,4 @@
     </visual>
     <collision>
-      <origin xyz="0 0 0" rpy="0 0 0"/>
       <geometry>
         <sphere radius="${caster_wheel_radius}"/>
@@ -125,5 +160,5 @@
     <origin xyz="${caster_wheel_joint_offset} 0 -${0.06+caster_wheel_radius}" rpy="0 0 0"/>
   </joint>
-  <joint name="imu_joint" type="fixed">
+  <!-- <joint name="imu_joint" type="fixed">
     <parent link="base_link" />
     <child link="imu" />
@@ -151,5 +186,5 @@
   </joint>
   <link name="camera" type="fixed">
-  </link>
+  </link> -->
 <gazebo reference="left_wheel">
   <mu1>1.0</mu1>

Commit message: Last update. Fix many issues, and update robot characteristics.

File: urdf/robaka_v2.xacro (robot description, xacro)
@@ -1,13 +1,15 @@
 <?xml version="1.0"?>
 <robot xmlns:xacro="http://www.ros.org/wiki/xacro" name="robaka_v2">
-  <xacro:property name="base_width" value="0.3"/>
-  <xacro:property name="base_len" value="0.4"/>
-  <xacro:property name="base_height" value="0.12"/>
+  <xacro:property name="base_width" value="0.46"/>
+  <xacro:property name="base_len" value="0.635"/>
+  <xacro:property name="base_height" value="0.1"/>
   <xacro:property name="wheel_radius" value="0.085"/>
   <xacro:property name="base_wheel_gap" value="0.02"/>
-  <xacro:property name="wheel_separation" value="0.31"/>
-  <xacro:property name="wheel_joint_offset" value="-0.107"/>
-  <xacro:property name="caster_wheel_radius" value="0.0375"/>
-  <xacro:property name="caster_wheel_joint_offset" value="0.12"/>
+  <xacro:property name="wheel_separation" value="0.47"/>
+  <xacro:property name="wheel_joint_offset_x" value="-0.2175"/>
+  <xacro:property name="wheel_joint_offset_z" value="0.0275"/>
+  <xacro:property name="caster_wheel_radius" value="0.05"/>
+  <xacro:property name="caster_wheel_joint_offset_x" value="0.2625"/>
+  <xacro:property name="caster_wheel_joint_offset_z" value="0.035"/>
   <xacro:include filename="$(find robaka)/urdf/robaka_v2_gazebo_plugins.xacro"/>
   <material name="blue">
@@ -67,5 +69,5 @@
   </link>
   <joint name="base_link_joint" type="fixed">
-    <origin xyz="0 0 ${wheel_radius + 0.005}" rpy="0 0 0" />
+    <origin xyz="0 0 ${wheel_radius + 0.0275}" rpy="0 0 0" />
     <parent link="base_footprint"/>
     <child link="base_link" />
@@ -98,5 +100,5 @@
       <parent link="base_link"/>
       <child link="${prefix}_wheel"/>
-      <origin xyz="${wheel_joint_offset} ${((base_width/2)+base_wheel_gap)*reflect} -0.06" rpy="0 0 0"/>
+      <origin xyz="${wheel_joint_offset_x} ${((base_width/2)+base_wheel_gap)*reflect} -${base_height/2 + wheel_joint_offset_z}" rpy="0 0 0"/>
     </joint>
   </xacro:macro>
@@ -129,5 +131,5 @@
     <parent link="base_link"/>
     <child link="caster_wheel"/>
-    <origin xyz="${caster_wheel_joint_offset} 0 -${0.06+caster_wheel_radius}" rpy="0 0 0"/>
+    <origin xyz="${caster_wheel_joint_offset_x} 0 -${caster_wheel_joint_offset_z+caster_wheel_radius + base_height/2}" rpy="0 0 0"/>
   </joint>
   <joint name="imu_joint" type="fixed">

Commit message: Fix issues

File: urdf/robaka_v2.xacro (robot description, xacro)
@@ -139,10 +139,10 @@
   </joint>
   <link name="imu" />
-  <joint name="lidar_joint" type="fixed">
+  <joint name="zed_joint" type="fixed">
     <parent link="base_link" />
-    <child link="lidar" />
+    <child link="zed" />
     <origin xyz="0.0 0.0 0.12" rpy="0 0 3.14159" />
   </joint>
-  <link name="lidar">
+  <link name="zed">
     <visual>
       <material name="blue" />

Commit message: fix more issues

File: urdf/robaka_v2.xacro (robot description, xacro)
@@ -39,5 +39,4 @@
     </inertial>
   </xacro:macro>
-  <link name="dummy"/>
   <link name="base_footprint">
     <xacro:box_inertia m="8" w="0.001" h="0.001" d="0.001"/>
@@ -50,8 +49,8 @@
     </visual>
   </link>
-  <joint name="dummy_joint" type="fixed">
-     <parent link="dummy"/>
-     <child link="base_footprint"/>
-     </joint>
+  <joint name="base_footprint_joint" type="fixed">
+    <parent link="base_footprint"/>
+    <child link="base_link" />
+  </joint>
   <link name="base_link">
     <xacro:box_inertia m="1" w="${base_len}" h="${base_width}" d="0.01"/>
